File: viparTester.kicad_pcb (KiCad board)
At the start: 2 copper layers, 55 x 35 mm, 24 parts, among them J1 Conn_01x03, J2 Conn_01x04, J3 Conn_01x02, J4 Conn_01x04, J5 Conn_01x06, U1 L78L33_TO92, U2 ATtiny13-20SSU

Commit message: gerbers and milling
Parts:
- C3, C4: footprint Capacitor_SMD:C_0603_1608Metric_Pad1.08x0.95mm_HandSolder -> Capacitor_SMD:C_1206_3216Metric_Pad1.33x1.80mm_HandSolder
- moved J2 9.43 mm to (146.3, 98.2)
- moved J4 8.11 mm to (138.8, 122.0)
- moved R1 7.50 mm to (126.1, 94.1), turned to 90 degrees
- moved D1 7.08 mm to (128.5, 94.1)
- moved C3 5.99 mm to (114.9, 117.5)
- moved D4 5.21 mm to (145.5, 106.2)
- moved D5 5.21 mm to (157.1, 106.2)
- moved R4 5.21 mm to (148.5, 106.3)
- moved R5 5.21 mm to (154.0, 106.3)
- moved J1 4.33 mm to (123.8, 122.0)
- moved J5 3.83 mm to (126.9, 115.2)
- moved C4 0.69 mm to (121.5, 105.4)
Routing:
- net +12V: track 113.5 -> 123.7 mm, vias 0 -> 1
- net Net-(J5-Pad5): track 29.6 -> 20.5 mm
- net /O2: track 9.29 -> 18.1 mm
- net /O1: track 8.33 -> 15.1 mm
- net Net-(C2-Pad1): track 38.1 -> 43.7 mm
- net /IN2: track 34.2 -> 28.8 mm
- net /EN2: track 6.58 -> 10.9 mm
- net Net-(J5-Pad3): track 11.5 -> 7.88 mm
- net /EN1: track 8.11 -> 11.5 mm
- net /IN1: track 24.7 -> 23.7 mm
- net GND: vias 0 -> 1
Other:
- outline, holes or cut-outs redrawn
- board text added: "12v"
- board text added: "GND"
