File: viparTester.sch (KiCad schematic (older format))
At the start: 24 parts, among them J1 Conn_01x03, J2 Conn_01x04, J3 Conn_01x02, J4 Conn_01x04, J5 Conn_01x06, U1 L78L33_TO92, U2 ATtiny13-20SSU

Commit message: gerbers and milling
Parts:
- C3, C4: footprint Capacitor_SMD:C_0603_1608Metric_Pad1.08x0.95mm_HandSolder -> Capacitor_SMD:C_1206_3216Metric_Pad1.33x1.80mm_HandSolder
Changed lines of the file:
@@
 F 0 "C4" H 6692 3096 50  0000 L CNN
 F 1 "0.1uF" H 6692 3005 50  0000 L CNN
-F 2 "Capacitor_SMD:C_0603_1608Metric_Pad1.08x0.95mm_HandSolder" H 6600 3050 50  0001 C CNN
+F 2 "Capacitor_SMD:C_1206_3216Metric_Pad1.33x1.80mm_HandSolder" H 6600 3050 50  0001 C CNN
 F 3 "~" H 6600 3050 50  0001 C CNN
 	1    6600 3050
@@
 F 0 "C3" H 5792 3296 50  0000 L CNN
 F 1 "0.1uF" H 5792 3205 50  0000 L CNN
-F 2 "Capacitor_SMD:C_0603_1608Metric_Pad1.08x0.95mm_HandSolder" H 5700 3250 50  0001 C CNN
+F 2 "Capacitor_SMD:C_1206_3216Metric_Pad1.33x1.80mm_HandSolder" H 5700 3250 50  0001 C CNN
 F 3 "~" H 5700 3250 50  0001 C CNN
 	1    5700 3250
